File: hardware/pcb/mlb/VIA1+VIA2+RTC+ADB.sch (KiCad schematic (older format))
At the start: 22 parts, among them J10 ADB_CONN, J9 ADB_CONN, Q3 2N3904, Y1 32.768KHz

Commit message: Fix errors found in review of the Macintosh SE/30 schematic redraw.
Page 1:

* DSACK*(0:1) (syntax)
* R-W* (inconsistent syntax)
* IPL different syntax
* PDS 38, C16M not grounded
* PDS 39, should be grounded

Page 2:

* RAAF*(8), RABF*(9), RAAF*(10), RABF*(10) (syntax)
* RCMUX* (syntax)
* ROM* missing page 3 indicator
* ROMSIMM1 GND 10, 30, 64
* ROMSIMM1 Incorrect +5V lines
* ROMSIMM1 Confusing bus line drawing angles makes connections look
  duplicated

Page 3:

* VIAIRQ2* (syntax)
* VIAIRQ1N (syntax, on GLUE template)
* SCCRD* (syntax)

Page 4:

* VIA template, RS0, RS1, RS2, RS3 erroneously written as R50, R51,
  R52, R53
* V1PB7 erroneously written as VIPB7
* RTC-D erroneously written as RTC-O
* V1PA0, V1PA1, V1PA2 erroneously written as VIPA0, VIPA1, VIPA2
* warning: additional label BATT not present
* UL11 ADB template, P5 erroneously written as P2
* ADBO erroneously written as ADB0
* SNDINT* erroneously written as SNTINT*

Page 5:

* HSYNC* on UG7 (syntax)
* UJ6 confusing bus line makes signals look duplicated
* Video ROM UK6 not labeled with reference designator (already inside
  KiCad file, stale PDF?)
* VIDS4, VIDS3, VIDS2, VIDS1, VIDS0 erroneously written a VID54,
  VID53, VID53, VID51, VID50
* R-W* alternate page reference erroneously written as RW*
* 74F253 template, G erroneously labeled as GND
* 74F253 template, missing second G enable pin
* style: C0 in 74F253 template should not be C0(GND)
* warning: UA8 ALTVID line could have another label close to the chip

Page 6:

* warning: On SWIM, WRDATA could have label WR*
* DB25 connector: DP*, DB0*, DB1*, DB2*, DB3*, DB4*, DB5*, DB6*, DB7*
  (syntax)
* J8 Ribbon Connector: Missing +12V on 13, 15, 17, 19
* J6 DB-19: Missing +12V-DSK on 7, 8
* warning: missing RDDATA.F additional label near J6 DB-19 pin 18
* warning: missing WRITE.F additional label near J6 DB-19 pin 19
* warning: confusing bus line layout on 53C80 looks like duplicate
  wiring

Page 7:

* RXDA+ erroneously written as RXDB+
* HSKOA erroneo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
Connections:
- net BATT: now reaches D1.2 (A)
- net ADB0 renamed ADBO
- net RTC-O renamed RTC-D
- net SNTINT* renamed SNDINT*
- net VIPA0 renamed V1PA0
- net VIPA1 renamed V1PA1
- net VIPA2 renamed V1PA2
- net VIPB7 renamed V1PB7
Changed lines of the file:
@@
 U 1 1 5EC1CBCA
 P 7500 5350
+AR Path="/5EC1CBCA" Ref="UL11"  Part="1"
+AR Path="/5EC6E211/5EC1CBCA" Ref="UL11"  Part="1"
 F 0 "UL11" H 7650 5400 50  0000 C CNN
 F 1 "ADB" H 7650 5300 50  0000 C CNN
@@
 $EndComp
 NoConn ~ 15950 -700
-Wire Wire Line
-	4300 1150 15800 1150
-Wire Wire Line
-	4300 1250 15800 1250
-Wire Wire Line
-	4300 1350 15800 1350
 Wire Wire Line
 	4300 1450 15800 1450
@@
 $EndComp
 Text Label 8500 4250 0    50   ~ 0
-RTC-O
+RTC-D
 Text Label 8500 4350 0    50   ~ 0
 RTC-CLK
@@
 	10700 6250 10900 6250
 Text Label 10750 5400 0    50   ~ 0
-ADB0
+ADBO
 Wire Wire Line
 	11150 5600 10900 5600
@@
 3.0V, 1/2AA
 Text Label 4350 1150 0    50   ~ 0
-VIPA0
+V1PA0
 Text Label 4350 1250 0    50   ~ 0
-VIPA1
+V1PA1
 Text Label 4350 1350 0    50   ~ 0
-VIPA2
+V1PA2
 Text Label 4350 1450 0    50   ~ 0
 SYNC
@@
 SCCWREQ*
 Text Label 4350 2050 0    50   ~ 0
-RTC-O
+RTC-D
 Text Label 4350 2150 0    50   ~ 0
 RTC-CLK
@@
 VSYNCEN*
 Text Label 4350 2750 0    50   ~ 0
-VIPB7
+V1PB7
 Text Label 4350 2950 0    50   ~ 0
 VIAIRQ1*
-Text GLabel 15800 1150 2    50   Input ~ 0
-VIPA0
-Text GLabel 15800 1250 2    50   Input ~ 0
-VIPA1
-Text GLabel 15800 1350 2    50   Input ~ 0
-VIPA2
 Text GLabel 15800 1450 2    50   Input ~ 0
 SYNC
@@
 VSYNCEN*
 Text GLabel 15800 2750 2    50   Input ~ 0
-VIPB7
+V1PB7
 Wire Wire Line
 	3300 3450 2900 3450
@@
 SCSIDRQ
 Text GLabel 1400 9550 0    50   Input ~ 0
-SNTINT*
+SNDINT*
 Text GLabel 1400 9650 0    50   Input ~ 0
 SCSIIRQ
@@
 Wire Bus Line
 	5350 7950 15800 7950
-Wire Bus Line
-	2300 1000 2300 7550
-Wire Bus Line
-	5350 7450 5350 7950
-Wire Bus Line
-	2450 1750 2450 8650
 Text Notes 1070 1035 2    50   ~ 0
 (1-3,5-7)
@@
 Text Notes 1025 9485 2    50   ~ 0
 (3)
-Text Notes 1055 9585 2    50   ~ 0
+Text Notes 1042 9586 2    50   ~ 0
 (7)
 Text Notes 1050 9685 2    50   ~ 0
 (6)
-Text Notes 16065 1180 0    50   ~ 0
-(8,9)
-Text Notes 16065 1280 0    50   ~ 0
-(8,9)
-Text Notes 16065 1380 0    50   ~ 0
-(8,9)
 Text Notes 16060 1480 0    50   ~ 0
 (3)
@@
 Text Notes 16225 2685 0    50   ~ 0
 (1)
-Text Notes 16065 2785 0    50   ~ 0
+Text Notes 16095 2781 0    50   ~ 0
 (9)
 Text GLabel 15800 2950 2    50   Input ~ 0
@@
 Text Notes 16175 9185 0    50   ~ 0
 (3)
+Wire Wire Line
+	4300 1350 15800 1350
+Wire Wire Line
+	4300 1250 15800 1250
+Wire Wire Line
+	4300 1150 15800 1150
+Text Notes 16090 1180 0    50   ~ 0
+(8,9)
+Text Notes 16090 1280 0    50   ~ 0
+(8,9)
+Text Notes 16090 1380 0    50   ~ 0
+(8,9)
+Text GLabel 15800 1350 2    50   Input ~ 0
+V1PA2
+Text GLabel 15800 1250 2    50   Input ~ 0
+V1PA1
+Text GLabel 15800 1150 2    50   Input ~ 0
+V1PA0
+Wire Bus Line
+	2300 1000 2300 7550
+Wire Bus Line
+	5350 7450 5350 7950
+Wire Bus Line
+	2450 1750 2450 8650
+Text Label 13900 3650 0    50   ~ 0
+BATT
 $EndSCHEMATC
